File: overvolt/overvolt.kicad_pcb (KiCad board)
At the start: 2 copper layers, 53.6 x 30.8 mm, 15 parts, among them J1 Output, J2 Input, Q1 2N6504D, U1 MC3423

Commit message: PCB in factory, lets see the first results
Parts:
- moved R1 0.60 mm to (125.4, 144.6)
- moved R3 0.60 mm to (121.8, 144.6)
Routing:
- net VCC: track 37.5 -> 48.2 mm
- net Net-(C1-Pad1): track 121.8 -> 125.1 mm
- net Net-(JP2-Pad2): track 6.87 -> 9.25 mm
- net GND: vias 14 -> 23
