File: overvolt.sch (KiCad schematic (older format))
At the start: 15 parts, among them J1 Output, J2 Input, Q1 2N6504D, U1 MC3423

Commit message: Repaired moving project
Parts:
- U1: symbol Connector:MC3423 -> overvolt-rescue:MC3423-Connector
Changed lines of the file:
@@
 $EndComp
 $Comp
-L Connector:MC3423 U1
+L overvolt-rescue:MC3423-Connector U1
 U 1 1 60B20B6F
 P 4700 2800
